Commit message: updated urdf with exact real world setup

File: robofin/urdf/franka_panda/panda_finray.urdf (robot description, URDF)
Before this commit: robot panda, 14 links, 13 joints
Links:
- added link camera; collision box size=0.042 0.023 .042; visual box size=0.042 0.023 .042
- added link camera_mount; collision mesh filename=mesh/camera/d405_mount.obj; visual mesh filename=mesh/camera/d405_mount.obj
- link panda_hand: geometry collision mesh filename=meshes/collision/hand.stl; visual mesh filename=meshes/visual/hand.dae
Joints:
- added joint camera_joint: type fixed, parent panda_hand, child camera_mount, origin xyz=0 0 0 rpy=1.57 0 -1.57
- added joint camera_joint2: type fixed, parent camera_mount, child camera, origin xyz=0 0 0 rpy=0 0 0
- joint panda_hand_joint: origin xyz=0 0 0 rpy=0 0 -0.785398163397 -> xyz=0 0 0.004 rpy=0 0 -0.785398163397

Commit message: added cube mesh and updated panda finray with masses and better colors

File: robofin/urdf/franka_panda/panda_finray.urdf (robot description, URDF)
Before this commit: robot panda, 16 links, 15 joints
Links:
- link camera: mass None -> 0.06; geometry collision mesh filename=mesh/camera/cube_mesh.obj; visual mesh filename=mesh/camera/cube_mesh.obj
- link camera_mount: mass None -> 0.023
- link panda_leftfinger: mass 0.1 -> 0.089
- link panda_rightfinger: mass 0.1 -> 0.089

Commit message: update urdf with correct mass and colors for visibility

File: robofin/urdf/franka_panda/panda_finray.urdf (robot description, URDF)
Before this commit: robot panda, 16 links, 15 joints
Links:
- link panda_leftfinger: mass 0.089 -> 0.081
- link panda_rightfinger: mass 0.089 -> 0.081

Commit message: camera mounts break the urdf

File: robofin/urdf/franka_panda/panda_finray.urdf (robot description, URDF)
Before this commit: robot panda, 16 links, 15 joints
Links:
- removed link camera
- removed link camera_mount
Joints:
- removed joint camera_joint
- removed joint camera_joint2

Commit message: franka shift by .004 since we removed the camera mount

File: robofin/urdf/franka_panda/panda_finray.urdf (robot description, URDF)
Before this commit: robot panda, 14 links, 13 joints
Joints:
- joint panda_hand_joint: origin xyz=0 0 0.004 rpy=0 0 -0.785398163397 -> xyz=0 0 0.0 rpy=0 0 -0.785398163397
